File: BasicPr/BasicPr.kicad_pcb (KiCad board)
At the start: 2 copper layers, 8 parts, among them U1 NE555P

Commit message: PCB Básica Final
Parts:
- C1: footprint Capacitor_THT:CP_Radial_D8.0mm_P3.80mm -> Capacitor_THT:CP_Radial_D5.0mm_P2.50mm
- moved D2 37.2 mm to (22.2, 43.5)
- moved U1 28.9 mm to (23.5, 30.5)
- moved C1 27.9 mm to (17.8, 31.7), turned to 90 degrees
- moved D1 26.0 mm to (28.6, 43.5)
- moved R4 22.6 mm to (17.8, 42.5), turned to 90 degrees
- moved R1 17.3 mm to (23.5, 25.4)
- moved R2 6.27 mm to (34.3, 31.1)
- moved R3 3.32 mm to (41.9, 33.7), turned to -90 degrees
Connections:
- net Net-(U1-DIS) renamed GND
Routing:
- net VCC: track 0.00 -> 45.2 mm
- net /THR: track 0.00 -> 22.2 mm
- net Net-(D1-A): track 0.00 -> 20.8 mm
- net Net-(D1-K): track 0.00 -> 15.1 mm
- net Net-(D2-K): track 0.00 -> 4.87 mm
- added copper zone on F.Cu, net GND
Other:
- board outline added: 31.1 x 27.9 mm
- board text added: ":D"
